File: Untitled.kicad_sch (KiCad schematic)
At the start: 3 parts, among them J1 USB_C_Receptacle_PowerOnly_6P

Commit message: FINSIHEDDD
Parts:
- removed J1: USB_C_Receptacle_PowerOnly_6P, Connector_USB:USB_C_Plug_JAE_DX07P024AJ1, symbol Connector:USB_C_Receptacle_PowerOnly_6P
- added J2: USB_C_Receptacle_PowerOnly_6P, Connector_USB:USB_C_Plug_smaller, symbol Connector:USB_C_Receptacle_PowerOnly_6P
Connections:
- net at D1.1 (K): now also J2.A12 (GND), J2.B12 (GND), J2.S1 (SHIELD)
- net at R1.1: now also J2.A9 (VBUS), J2.B9 (VBUS)
Other:
- moved on the sheet: D1, R1
Changed lines of the file:
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@@
 	(paper "A4")
 	(junction
-		(at 114.3 99.06)
+		(at 97.79 91.44)
 		(diameter 0)
 		(color 0 0 0 0)
 	)
+	(junction
+		(at 113.03 64.77)
+		(diameter 0)
+		(color 0 0 0 0)
+	)
 	(no_connect
-		(at 129.54 85.09)
+		(at 113.03 80.01)
 	)
 	(no_connect
-		(at 129.54 82.55)
-	)
-	(wire
-		(pts
-			(xy 147.32 77.47) (xy 147.32 69.85)
-		)
-		(stroke
-			(width 0)
-			(type default)
-		)
-	)
-	(wire
-		(pts
-			(xy 106.68 99.06) (xy 114.3 99.06)
-		)
-		(stroke
-			(width 0)
-			(type default)
-		)
-	)
-	(wire
-		(pts
-			(xy 147.32 86.36) (xy 147.32 85.09)
-		)
-		(stroke
-			(width 0)
-			(type default)
-		)
-	)
-	(wire
-		(pts
-			(xy 106.68 95.25) (xy 106.68 99.06)
-		)
-		(stroke
-			(width 0)
-			(type default)
-		)
-	)
-	(wire
-		(pts
-			(xy 147.32 69.85) (xy 129.54 69.85)
-		)
-		(stroke
-			(width 0)
-			(type default)
-		)
-	)
-	(wire
-		(pts
-			(xy 147.32 99.06) (xy 147.32 93.98)
-		)
-		(stroke
-			(width 0)
-			(type default)
-		)
-	)
-	(wire
-		(pts
-			(xy 114.3 95.25) (xy 114.3 99.06)
-		)
-		(stroke
-			(width 0)
-			(type default)
-		)
-	)
-	(wire
-		(pts
-			(xy 114.3 99.06) (xy 147.32 99.06)
+		(at 113.03 77.47)
+	)
+	(wire
+		(pts
+			(xy 147.32 68.58) (xy 147.32 72.39)
+		)
+		(stroke
+			(width 0)
+			(type default)
+		)
+	)
+	(wire
+		(pts
+			(xy 90.17 90.17) (xy 90.17 91.44)
+		)
+		(stroke
+			(width 0)
+			(type default)
+		)
+	)
+	(wire
+		(pts
+			(xy 147.32 81.28) (xy 147.32 80.01)
+		)
+		(stroke
+			(width 0)
+			(type default)
+		)
+	)
+	(wire
+		(pts
+			(xy 90.17 91.44) (xy 97.79 91.44)
+		)
+		(stroke
+			(width 0)
+			(type default)
+		)
+	)
+	(wire
+		(pts
+			(xy 147.32 91.44) (xy 147.32 88.9)
+		)
+		(stroke
+			(width 0)
+			(type default)
+		)
+	)
+	(wire
+		(pts
+			(xy 113.03 68.58) (xy 147.32 68.58)
+		)
+		(stroke
+			(width 0)
+			(type default)
+		)
+	)
+	(wire
+		(pts
+			(xy 97.79 91.44) (xy 147.32 91.44)
+		)
+		(stroke
+			(width 0)
+			(type default)
+		)
+	)
+	(wire
+		(pts
+			(xy 97.79 90.17) (xy 97.79 91.44)
+		)
+		(stroke
+			(width 0)
+			(type default)
+		)
+	)
+	(wire
+		(pts
+			(xy 113.03 64.77) (xy 113.03 68.58)
 		)
 		(stroke
@@
 	(symbol
 		(lib_id "Connector:USB_C_Receptacle_PowerOnly_6P")
-		(at 114.3 77.47 0)
+		(at 97.79 72.39 0)
 		(unit 1)
 		(exclude_from_sim no)
@@
 		(dnp no)
 		(fields_autoplaced yes)
-		(property "Reference" "J1"
-			(at 114.3 59.69 0)
+		(property "Reference" "J2"
+			(at 97.79 54.61 0)
 			(effects
 				(font
@@
 		)
 		(property "Value" "USB_C_Receptacle_PowerOnly_6P"
-			(at 114.3 62.23 0)
-			(effects
-				(font
-					(size 1.27 1.27)
-				)
-			)
-		)
-		(property "Footprint" "Connector_USB:USB_C_Plug_JAE_DX07P024AJ1"
-			(at 118.11 74.93 0)
+			(at 97.79 57.15 0)
+			(effects
+				(font
+					(size 1.27 1.27)
+				)
+			)
+		)
+		(property "Footprint" "Connector_USB:USB_C_Plug_smaller"
+			(at 101.6 69.85 0)
 			(effects
 				(font
@@
 		)
 		(property "Datasheet" "https://www.usb.org/sites/default/files/documents/usb_type-c.zip"
-			(at 114.3 77.47 0)
+			(at 97.79 72.39 0)
 			(effects
 				(font
@@
 		)
 		(property "Description" "USB Power-Only 6P Type-C Receptacle connector"
-			(at 114.3 77.47 0)
+			(at 97.79 72.39 0)
 			(effects
 				(font
@@
 		(pin "B12"
 		)
+		(pin "S1"
+		)
 		(pin "A12"
-		)
-		(pin "S1"
 		)
 		(instances
 			(project "Untitled"
 				(path "/b037e26d-df73-4092-bdd1-a95aa78e379c"
-					(reference "J1")
+					(reference "J2")
+					(unit 1)
+				)
+			)
+		)
+	)
+	(symbol
+		(lib_id "power:PWR_FLAG")
+		(at 113.03 64.77 0)
+		(unit 1)
+		(exclude_from_sim no)
+		(in_bom yes)
+		(on_board yes)
+		(dnp no)
+		(fields_autoplaced yes)
+		(property "Reference" "#FLG01"
+			(at 113.03 62.865 0)
+			(effects
+				(font
+					(size 1.27 1.27)
+				)
+				(hide yes)
+			)
+		)
+		(property "Value" "PWR_FLAG"
+			(at 113.03 59.69 0)
+			(effects
+				(font
+					(size 1.27 1.27)
+				)
+			)
+		)
+		(property "Footprint" ""
+			(at 113.03 64.77 0)
+			(effects
+				(font
+					(size 1.27 1.27)
+				)
+				(hide yes)
+			)
+		)
+		(property "Datasheet" "~"
+			(at 113.03 64.77 0)
+			(effects
+				(font
+					(size 1.27 1.27)
+				)
+				(hide yes)
+			)
+		)
+		(property "Description" "Special symbol for telling ERC where power comes from"
+			(at 113.03 64.77 0)
+			(effects
+				(font
+					(size 1.27 1.27)
+				)
+				(hide yes)
+			)
+		)
+		(pin "1"
+		)
+		(instances
+			(project "Untitled"
+				(path "/b037e26d-df73-4092-bdd1-a95aa78e379c"
+					(reference "#FLG01")
 					(unit 1)
 				)
@@
 	(symbol
 		(lib_id "Device:R")
-		(at 147.32 81.28 0)
+		(at 147.32 76.2 0)
 		(unit 1)
 		(exclude_from_sim no)
@@
 		(fields_autoplaced yes)
 		(property "Reference" "R1"
-			(at 149.86 80.0099 0)
+			(at 149.86 74.9299 0)
 			(effects
 				(font
@@
 		)
 		(property "Value" "R"
-			(at 149.86 82.5499 0)
+			(at 149.86 77.4699 0)
 			(effects
 				(font
@@
 		)
 		(property "Footprint" "Resistor_SMD:R_01005_0402Metric"
-			(at 145.542 81.28 90)
+			(at 145.542 76.2 90)
 			(effects
 				(font
@@
 		)
 		(property "Datasheet" "~"
-			(at 147.32 81.28 0)
+			(at 147.32 76.2 0)
 			(effects
 				(font
@@
 		)
 		(property "Description" "Resistor"
-			(at 147.32 81.28 0)
+			(at 147.32 76.2 0)
 			(effects
 				(font
@@
 	(symbol
 		(lib_id "Device:LED")
-		(at 147.32 90.17 90)
+		(at 147.32 85.09 90)
 		(unit 1)
 		(exclude_from_sim no)
@@
 		(fields_autoplaced yes)
 		(property "Reference" "D1"
-			(at 151.13 90.4874 90)
+			(at 151.13 85.4074 90)
 			(effects
 				(font
@@
 		)
 		(property "Value" "LED"
-			(at 151.13 93.0274 90)
+			(at 151.13 87.9474 90)
 			(effects
 				(font
@@
 		)
 		(property "Footprint" "LED_SMD:LED_RGB_1210"
-			(at 147.32 90.17 0)
+			(at 147.32 85.09 0)
 			(effects
 				(font
@@
 		)
 		(property "Datasheet" "~"
-			(at 147.32 90.17 0)
+			(at 147.32 85.09 0)
 			(effects
 				(font
@@
 		)
 		(property "Description" "Light emitting diode"
-			(at 147.32 90.17 0)
+			(at 147.32 85.09 0)
 			(effects
 				(font
@@
 		)
 		(property "Sim.Pins" "1=K 2=A"
-			(at 147.32 90.17 0)
-			(effects
-				(font
+			(at 147.32 85.09 0)
+			(effects
+				(font
